File: pcb/roller/ecu/05_Security.kicad_sch (KiCad schematic)
At the start: 19 parts, among them Q6 2N7002KQ-7, U300 SN74AHCT541QPWRQ1, U301 TPIC6A595DWR, U302 TPIC6A595DWR, U303 TPIC6A595DWR, U304 TPIC6A595DWR

Commit message: Add design settings and DRC rules to ECU PCB configuration
- Introduced comprehensive design settings including defaults for various parameters such as line widths, text sizes, and pad dimensions.
- Added detailed DRC (Design Rule Check) exclusions and rule severities to enhance error handling and warnings during PCB design.
- Updated tuning pattern settings and teardrop parameters for improved track and pad connections.
- Cleared previously used designators for better organization and clarity in the design file.
Parts:
- U301, U302, U303, U304: symbol ECU_Custom:TPIC6A595DWR -> Starlight:TPIC6A595DWR
Other:
- note added: "PE2"
- note added: "PE3"
- note added: "PE4"
- note added: "PE5"
- note added: "PE6"
- note added: "PE7"
Changed lines of the file:
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@@
 	(generator_version "10.0")
 	(paper "A4")
+	(text "PE7"
+		(exclude_from_sim no)
+		(at 39.37 175.26 0)
+		(effects
+			(font
+				(size 1.27 1.27)
+			)
+			(justify right bottom)
+		)
+	)
+	(text "PE4"
+		(exclude_from_sim no)
+		(at 80.01 140.97 0)
+		(effects
+			(font
+				(size 1.27 1.27)
+			)
+			(justify right bottom)
+		)
+	)
+	(text "PE2"
+		(exclude_from_sim no)
+		(at 80.01 138.43 0)
+		(effects
+			(font
+				(size 1.27 1.27)
+			)
+			(justify right bottom)
+		)
+	)
+	(text "PE5"
+		(exclude_from_sim no)
+		(at 80.01 143.51 0)
+		(effects
+			(font
+				(size 1.27 1.27)
+			)
+			(justify right bottom)
+		)
+	)
+	(text "PE6"
+		(exclude_from_sim no)
+		(at 80.01 135.89 0)
+		(effects
+			(font
+				(size 1.27 1.27)
+			)
+			(justify right bottom)
+		)
+	)
+	(text "PE3"
+		(exclude_from_sim no)
+		(at 80.01 146.05 0)
+		(effects
+			(font
+				(size 1.27 1.27)
+			)
+			(justify right bottom)
+		)
+	)
 	(junction
 		(at 185.42 90.17)
@@
 		)
 	)
-	(label "PE7"
-		(at 39.37 175.26 180)
-		(effects
-			(font
-				(size 1.27 1.27)
-			)
-			(justify right bottom)
-		)
-	)
 	(label "TPIC5_SRCK"
 		(at 43.18 100.33 0)
@@
 		)
 	)
-	(label "PE4"
-		(at 80.01 140.97 180)
-		(effects
-			(font
-				(size 1.27 1.27)
-			)
-			(justify right bottom)
-		)
-	)
 	(label "TPIC5_OE_N"
 		(at 43.18 85.09 0)
@@
 		)
 	)
-	(label "PE2"
-		(at 80.01 138.43 180)
-		(effects
-			(font
-				(size 1.27 1.27)
-			)
-			(justify right bottom)
-		)
-	)
-	(label "PE5"
-		(at 80.01 143.51 180)
-		(effects
-			(font
-				(size 1.27 1.27)
-			)
-			(justify right bottom)
-		)
-	)
 	(label "TPIC5_OE_N"
 		(at 161.29 146.05 180)
@@
 		)
 	)
-	(label "PE6"
-		(at 80.01 135.89 180)
-		(effects
-			(font
-				(size 1.27 1.27)
-			)
-			(justify right bottom)
-		)
-	)
 	(label "TPIC5_CLR_N"
 		(at 43.18 82.55 0)
@@
 		)
 	)
-	(label "PE3"
-		(at 80.01 146.05 180)
-		(effects
-			(font
-				(size 1.27 1.27)
-			)
-			(justify right bottom)
-		)
-	)
 	(label "TPIC5_SRCK"
 		(at 175.26 100.33 0)
@@
 	)
 	(symbol
-		(lib_id "ECU_Custom:TPIC6A595DWR")
+		(lib_id "Starlight:TPIC6A595DWR")
 		(at 82.55 91.44 0)
 		(unit 1)
@@
 	)
 	(symbol
-		(lib_id "ECU_Custom:TPIC6A595DWR")
+		(lib_id "Starlight:TPIC6A595DWR")
 		(at 82.55 41.91 0)
 		(unit 1)
@@
 	)
 	(symbol
-		(lib_id "ECU_Custom:TPIC6A595DWR")
+		(lib_id "Starlight:TPIC6A595DWR")
 		(at 214.63 91.44 0)
 		(unit 1)
@@
 	)
 	(symbol
-		(lib_id "ECU_Custom:TPIC6A595DWR")
+		(lib_id "Starlight:TPIC6A595DWR")
 		(at 214.63 39.37 0)
 		(unit 1)
