File: pcb/roller/ecu/07_Valve.kicad_sch (KiCad schematic)
At the start: 22 parts, among them Q2 NVD5C684NLT4G, Q3 NVD5C684NLT4G, U10 UCC27517AQDBVRQ1, U11 UCC27517AQDBVRQ1, U12 INA240A1D, U6 INA240A1D

Commit message: Add design settings and DRC rules to ECU PCB configuration
- Introduced comprehensive design settings including defaults for various parameters such as line widths, text sizes, and pad dimensions.
- Added detailed DRC (Design Rule Check) exclusions and rule severities to enhance error handling and warnings during PCB design.
- Updated tuning pattern settings and teardrop parameters for improved track and pad connections.
- Cleared previously used designators for better organization and clarity in the design file.
Connections:
- net +12V renamed YV_BACK_COIL_P
- net YV_BACK_COIL_P: no longer D2.1 (K)
- new net YV_FWD_COIL_P: D2.1 (K)
Other:
- note added: "PA4"
- note added: "PA6"
- note added: "PB6"
- note added: "PB7"
