File: pcb/roller/ecu/06_Relay.kicad_sch (KiCad schematic)
At the start: 31 parts, among them K1 Relay_SPDT, K10 Relay_SPST-NO, K11 Relay_SPDT, K12 Relay_SPDT, K13 Relay_SPDT, K14 Relay_SPST-NO, K15 Relay_SPST-NO, K16 Relay_SPST-NO, K17 Relay_SPST-NO, K18 Relay_SPST-NO, K19 Relay_SPST-NO, K2 Relay_SPDT, K20 Relay_SPST-NO, K21 Relay_SPST-NO, K22 Relay_SPST-NO, K23 Relay_SPST-NO, K24 Relay_SPDT, K25 Relay_SPST-NO, K26 Relay_SPST-NO, K27 Relay_SPST-NO, K3 Relay_SPDT, K4 Relay_SPST-NO, K5 Relay_SPDT, K6 Relay_SPST-NO, K7 Relay_SPDT, K8 Relay_SPST-NO, K9 Relay_SPDT

Commit message: Add ESTOP_NC pin and wire connections in ECU schematic; update designators in PCB project
Connections:
- net +12V: no longer K10.14, K12.A1, K17.14, K18.14, K19.14, K22.14, K24.14, K4.14, K6.14, K8.14
- new net +BAT: K10.14, K17.14, K18.14, K19.14, K22.14, K24.14, K4.14, K6.14, K8.14
- new net ESTOP_NC: K12.A1

Commit message: Refactor ECU schematic and project files
- Updated used designators in ecu.kicad_pro to reflect current components.
- Adjusted wire connections in ecu.kicad_sch for better layout and clarity.
- Added new wires and labels for ESTOP functionality.
- Modified pin placements and sizes for improved organization in the schematic.
- Ensured all changes maintain compatibility with existing design specifications.
Parts:
- removed K12: Relay_SPDT, Starlight:Relay_SPDT_Hongfa_HFV6_1FormC, symbol Relay:Relay_SPDT
- added K12: Relay_SPST-NO, Starlight:Relay_SPST-NO_Hongfa_HFV6_1FormA, symbol Relay:Relay_SPST-NO
Connections:
- net ESTOP_NC: now also K12.A1
- net E_STOP_DEVICE_SIDE: now also K12.13
- net E_STOP_OEM_SIDE: now also K12.14
- net E_STOP_OVR_RLY_COIL_DRV: now also K12.A2
- no-connect marks 3 -> 2
Changed lines of the file:
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@@
 	)
 	(no_connect
-		(at 196.85 107.95)
-	)
-	(no_connect
 		(at 71.12 48.26)
 	)
@@
 	(wire
 		(pts
-			(xy 199.39 102.87) (xy 196.85 102.87)
+			(xy 199.39 107.95) (xy 196.85 107.95)
 		)
 		(stroke
@@
 	(hierarchical_label "E_STOP_OEM_SIDE"
 		(shape input)
-		(at 199.39 102.87 0)
+		(at 199.39 107.95 0)
 		(effects
 			(font
@@
 	)
 	(symbol
-		(lib_id "Relay:Relay_SPDT")
-		(at 189.23 100.33 270)
-		(unit 1)
-		(body_style 1)
-		(exclude_from_sim no)
-		(in_bom yes)
-		(on_board yes)
-		(in_pos_files yes)
-		(dnp no)
-		(fields_autoplaced yes)
-		(property "Reference" "K12"
-			(at 189.23 85.09 90)
-			(show_name no)
-			(do_not_autoplace no)
-			(effects
-				(font
-					(size 1.27 1.27)
-				)
-			)
-		)
-		(property "Value" "Relay_SPDT"
-			(at 189.23 87.63 90)
-			(show_name no)
-			(do_not_autoplace no)
-			(effects
-				(font
-					(size 1.27 1.27)
-				)
-			)
-		)
-		(property "Footprint" "Starlight:Relay_SPDT_Hongfa_HFV6_1FormC"
-			(at 187.96 111.76 0)
-			(hide yes)
-			(show_name no)
-			(do_not_autoplace no)
-			(effects
-				(font
-					(size 1.27 1.27)
-				)
-				(justify left)
-			)
-		)
-		(property "Datasheet" ""
-			(at 189.23 100.33 0)
-			(hide yes)
-			(show_name no)
-			(do_not_autoplace no)
-			(effects
-				(font
-					(size 1.27 1.27)
-				)
-			)
-		)
-		(property "Description" "Relay SPDT, monostable, EN50005"
-			(at 189.23 100.33 0)
-			(hide yes)
-			(show_name no)
-			(do_not_autoplace no)
-			(effects
-				(font
-					(size 1.27 1.27)
-				)
-			)
-		)
-		(pin "A1"
-		)
-		(pin "A2"
-		)
-		(pin "14"
-		)
-		(pin "12"
-		)
-		(pin "11"
-		)
-		(instances
-			(project "ecu"
-				(path "/e5f3c8f3-31b1-4864-b028-38bb5e50c369/8ecbc12a-0669-48e9-8a42-e12d90c95eca"
-					(reference "K12")
-					(unit 1)
-				)
-			)
-		)
-	)
-	(symbol
 		(lib_id "power:+12V")
 		(at 204.47 171.45 0)
@@
 					(unit 1)
 				)
+			)
+		)
+	)
+	(symbol
+		(lib_id "Relay:Relay_SPST-NO")
+		(at 189.23 100.33 270)
+		(unit 1)
+		(body_style 1)
+		(exclude_from_sim no)
+		(in_bom yes)
+		(on_board yes)
+		(in_pos_files yes)
+		(dnp no)
+		(fields_autoplaced yes)
+		(property "Reference" "K12"
+			(at 189.23 85.09 90)
+			(show_name no)
+			(do_not_autoplace no)
+			(effects
+				(font
+					(size 1.27 1.27)
+				)
+			)
+		)
+		(property "Value" "Relay_SPST-NO"
+			(at 189.23 87.63 90)
+			(show_name no)
+			(do_not_autoplace no)
+			(effects
+				(font
+					(size 1.27 1.27)
+				)
+			)
+		)
+		(property "Footprint" "Starlight:Relay_SPST-NO_Hongfa_HFV6_1FormA"
+			(at 187.96 111.76 0)
+			(hide yes)
+			(show_name no)
+			(do_not_autoplace no)
+			(effects
+				(font
+					(size 1.27 1.27)
+				)
+				(justify left)
+			)
+		)
+		(property "Datasheet" ""
+			(at 189.23 100.33 0)
+			(hide yes)
+			(show_name no)
+			(do_not_autoplace no)
+			(effects
+				(font
+					(size 1.27 1.27)
+				)
+			)
+		)
+		(property "Description" "Relay SPST, normally open, EN50005"
+			(at 189.23 100.33 0)
+			(hide yes)
+			(show_name no)
+			(do_not_autoplace no)
+			(effects
+				(font
+					(size 1.27 1.27)
+				)
+			)
+		)
+		(pin "A1"
+		)
+		(pin "13"
+		)
+		(pin "14"
+		)
+		(pin "A2"
+		)
+		(instances
+			(project "ecu"
+				(path "/e5f3c8f3-31b1-4864-b028-38bb5e50c369/8ecbc12a-0669-48e9-8a42-e12d90c95eca"
+					(reference "K12")
+					(unit 1)
+				)

Commit message: Implement code changes to enhance functionality and improve performance
Connections:
- net +12V: no longer K20.14
- net +BAT: now also K20.14
Changed lines of the file:
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@@
+	)
+	(symbol
+		(lib_id "power:+BATT")
+		(at 203.2 46.99 0)
+		(unit 1)
+		(body_style 1)
+		(exclude_from_sim no)
+		(in_bom yes)
+		(on_board yes)
+		(in_pos_files yes)
+		(dnp no)
+		(fields_autoplaced yes)
+		(property "Reference" "#PWR0131"
+			(at 203.2 50.8 0)
+			(hide yes)
+			(show_name no)
+			(do_not_autoplace no)
+			(effects
+				(font
+					(size 1.27 1.27)
+				)
+			)
+		)
+		(property "Value" "+BAT"
+			(at 203.2 41.91 0)
+			(show_name no)
+			(do_not_autoplace no)
+			(effects
+				(font
+					(size 1.27 1.27)
+				)
+			)
+		)
+		(property "Footprint" ""
+			(at 203.2 46.99 0)
+			(hide yes)
+			(show_name no)
+			(do_not_autoplace no)
+			(effects
+				(font
+					(size 1.27 1.27)
+				)
+			)
+		)
+		(property "Datasheet" ""
+			(at 203.2 46.99 0)
+			(hide yes)
+			(show_name no)
+			(do_not_autoplace no)
+			(effects
+				(font
+					(size 1.27 1.27)
+				)
+			)
+		)
+		(property "Description" "Power symbol creates a global label with name \"+BATT\""
+			(at 203.2 46.99 0)
+			(hide yes)
+			(show_name no)
+			(do_not_autoplace no)
+			(effects
+				(font
+					(size 1.27 1.27)
+				)
+			)
+		)
+		(pin "1"
+		)
+		(instances
+			(project "ecu"
+				(path "/e5f3c8f3-31b1-4864-b028-38bb5e50c369/8ecbc12a-0669-48e9-8a42-e12d90c95eca"
+					(reference "#PWR0131")
+					(unit 1)
+				)
+			)
+		)
 	)
 	(symbol
@@
 					(unit 1)
 				)
-			)
-		)
-	)
-	(symbol
-		(lib_id "power:+12V")
-		(at 203.2 46.99 0)
-		(unit 1)
-		(body_style 1)
-		(exclude_from_sim no)
-		(in_bom yes)
-		(on_board yes)
-		(in_pos_files yes)
-		(dnp no)
-		(fields_autoplaced yes)
-		(property "Reference" "#PWR0134"
-			(at 203.2 50.8 0)
-			(hide yes)
-			(show_name no)
-			(do_not_autoplace no)
-			(effects
-				(font
-					(size 1.27 1.27)
-				)
-			)
-		)
-		(property "Value" "+12V"
-			(at 203.2 41.91 0)
-			(show_name no)
-			(do_not_autoplace no)
-			(effects
-				(font
-					(size 1.27 1.27)
-				)
-			)
-		)
-		(property "Footprint" ""
-			(at 203.2 46.99 0)
-			(hide yes)
-			(show_name no)
-			(do_not_autoplace no)
-			(effects
-				(font
-					(size 1.27 1.27)
-				)
-			)
-		)
-		(property "Datasheet" ""
-			(at 203.2 46.99 0)
-			(hide yes)
-			(show_name no)
-			(do_not_autoplace no)
-			(effects
-				(font
-					(size 1.27 1.27)
-				)
-			)
-		)
-		(property "Description" "Power symbol creates a global label with name \"+12V\""
-			(at 203.2 46.99 0)
-			(hide yes)
-			(show_name no)
-			(do_not_autoplace no)
-			(effects
-				(font
-					(size 1.27 1.27)
-				)
-			)
-		)
-		(pin "1"
-		)
-		(instances
-			(project "ecu"
-				(path "/e5f3c8f3-31b1-4864-b028-38bb5e50c369/8ecbc12a-0669-48e9-8a42-e12d90c95eca"
-					(reference "#PWR0134")
-					(unit 1)
-				)
