File: pcb/roller/ecu/02_MCU_Core.kicad_sch (KiCad schematic)
At the start: 36 parts, among them J1 SWD, SW1 SW_Push, U1 STM32H563ZITx, U221 ATECC608C-SSHDA-T, Y1 32.768kHz, Y2 25MHz

Commit message: Add power symbols for +1V0 and PWR_FLAG to the schematic
- Introduced a new global power symbol for +1V0 with appropriate properties and pin configurations.
- Added a PWR_FLAG symbol to indicate power source in the schematic, enhancing ERC capabilities.
- Updated the used designators in the project file to include new power symbols.
Parts:
- C41, C42: value 100nF -> 2.2uF
Connections:
- net +3.3V: now also U1.106 (VDDUSB), U1.108 (VDD), U1.121 (VDDIO2), U1.131 (VDD), U1.144 (VDD), U1.17 (VDD), U1.30 (VDD), U1.39 (VDD), U1.52 (VDD), U1.62 (VDD), U1.72 (VDD), U1.84 (VDD), U1.95 (VDD)
- net at C41.1, U1.142 (VCAP): no longer C42.1, U1.70 (VCAP)
- new net: C42.1, U1.70 (VCAP)
Other:
- moved on the sheet: C41, C42

Commit message: Add design settings and DRC rules to ECU PCB configuration
- Introduced comprehensive design settings including defaults for various parameters such as line widths, text sizes, and pad dimensions.
- Added detailed DRC (Design Rule Check) exclusions and rule severities to enhance error handling and warnings during PCB design.
- Updated tuning pattern settings and teardrop parameters for improved track and pad connections.
- Cleared previously used designators for better organization and clarity in the design file.
Parts:
- removed C40: 1uF, Capacitor_SMD:C_0603_1608Metric, symbol Device:C
- U221: symbol ECU_Custom:ATECC608C-SSHDA-T -> Starlight:ATECC608C-SSHDA-T
Connections:
- net PB8 renamed SAFE_I2C_SCL
- net PB9 renamed SAFE_I2C_SDA
Other:
- note added: "PA0"
- note added: "PA1"
- note added: "PA2"
- note added: "PA4"
- note added: "PA6"
- note added: "PA7"
- note added: "PB0"
- note added: "PB1"
- note added: "PB12"
- note added: "PB13"
- note added: "PB14"
- note added: "PB15"
- note added: "PB6"
- note added: "PB7"
- note added: "PB8"
- note added: "PB9"
- note added: "PC0"
- note added: "PC1"
- note added: "PC2"
- note added: "PC3"
- note added: "PC4"
- note added: "PC5"
- note added: "PD0"
- note added: "PD1"
- note added: "PE2"
- note added: "PE3"
- note added: "PE4"
- note added: "PE5"
- note added: "PE6"
- note added: "PE7"
- note added: "PG11"
- note added: "PG13"

Commit message: Add ESTOP_NC pin and wire connections in ECU schematic; update designators in PCB project
Parts:
- added R105, R106: 2.2k, Resistor_SMD:R_0603_1608Metric, symbol Device:R
Connections:
- net +3.3V: now also R105.1, R106.1
- net SAFE_I2C_SCL: now also R106.2
- net SAFE_I2C_SDA: now also R105.2
- net TEMP1_NTC_ADC: now reaches U1.37 (PA3)
- net TEMP2_NTC_ADC: now reaches U1.41 (PA5)
- no-connect marks 74 -> 72
Other:
- note added: "PA3"
- note added: "PA5"
- moved on the sheet: C6, U221

Commit message: Refactor ECU schematic and project files
- Updated used designators in ecu.kicad_pro to reflect current components.
- Adjusted wire connections in ecu.kicad_sch for better layout and clarity.
- Added new wires and labels for ESTOP functionality.
- Modified pin placements and sizes for improved organization in the schematic.
- Ensured all changes maintain compatibility with existing design specifications.
Connections:
- net ESTOP_DETECT: now reaches U1.48 (PB2)
- no-connect marks 72 -> 71
Other:
- note added: "PB2"

Commit message: Enhance ECU design files with updated parameters and new libraries
- Updated `ecu.kicad_pro` with new zone parameters, track widths, and DRC rules to improve design flexibility and manufacturability.
- Added `erc_report.json` to capture electrical rule check results, including warnings for multiple net names.
- Introduced `fp-lib-table` and `sym-lib-table` to include project-local libraries for footprints and symbols, enhancing design organization and accessibility.
Parts:
- D1: value ESDALC6V1-1U2 -> PESD5V0S1BA,115; footprint Diode_SMD:Infineon_SG-WLL-2-3_0.58x0.28_P0.36mm -> Diode_SMD:D_SOD-323; symbol Diode:ESD131-B1-W0201 -> Starlight:PESD5V0S1BA_115
