File: pcb/roller/ecu/ecu.kicad_pcb (KiCad board)
At the start: 4 copper layers, 187.6 x 139.6 mm, 275 parts, among them J1 SWD, J2 NTC, J3 SS-12400-004, J4 NTC, J6 TE-776163-1, J7 TE-776087-1, K1 Relay_SPDT, K10 Relay_SPST-NO, K11 Relay_SPDT, K12 Relay_SPST-NO, K13 Relay_SPDT, K14 Relay_SPST-NO, K15 Relay_SPST-NO, K16 Relay_SPST-NO, K17 Relay_SPST-NO, K18 Relay_SPST-NO, K19 Relay_SPST-NO, K2 Relay_SPDT, K20 Relay_SPST-NO, K21 Relay_SPST-NO, K22 Relay_SPST-NO, K23 Relay_SPST-NO, K24 Relay_SPDT, K25 Relay_SPST-NO, K26 Relay_SPST-NO, K27 Relay_SPST-NO, K3 Relay_SPDT, K4 Relay_SPST-NO, K5 Relay_SPDT, K6 Relay_SPST-NO, K7 Relay_SPDT, K8 Relay_SPST-NO, K9 Relay_SPDT, Q1 BSN20, Q2 NVD5C684NLT4G, Q3 NVD5C684NLT4G, Q4 BC817, Q5 BSC065N06LS5, Q6 2N7002KQ-7, Q9 BSN20, SW1 SW_Push, T201 KMS-1102NL, U1 STM32H563ZITx, U10 UCC27517AQDBVRQ1, U11 UCC27517AQDBVRQ1, U12 INA240A1D, U13 SN65HVD230, U14 SN65HVD230, U15 ACPL-214-500E, U2 LM74700, U221 ATECC608C-SSHDA-T, U300 SN74AHCT541QPWRQ1, U301 TPIC6A595DWR, U302 TPIC6A595DWR, U303 TPIC6A595DWR, U304 TPIC6A595DWR, U4 LAN8742A, U5 USBLC6-4SC6, U6 INA240A1D, U7 SN74LVC1G14DBV, U8 MPQ4371GVE-1000-AEC1-P, U9 MPQ2178GQHE-AEC1-Z, Y1 32.768kHz, Y2 25MHz, Y3 25MHz

Commit message: Implement code changes to enhance functionality and improve performance
Parts:
- moved R1 366.4 mm to (110.3, 118.1)
- moved C72 362.1 mm to (109.9, 123.0), turned to 0 degrees
- moved C74 362.0 mm to (116.5, 114.3), turned to 0 degrees
- moved C73 361.3 mm to (113.2, 123.0), turned to 0 degrees
- moved R80 359.9 mm to (122.4, 104.4)
- moved R79 359.2 mm to (120.6, 104.4)
- moved R2 354.3 mm to (127.5, 118.1)
- moved U10 353.1 mm to (121.9, 100.9), turned to 0 degrees
- moved C75 352.6 mm to (127.1, 123.0), turned to 0 degrees
- moved Q2 350.6 mm to (114.8, 102.7), turned to 0 degrees
- moved R81 349.9 mm to (124.2, 104.4)
- moved D2 347.8 mm to (113.3, 109.9), turned to 0 degrees
- moved C77 341.9 mm to (133.7, 114.3), turned to 0 degrees
- moved Q3 341.8 mm to (132.0, 102.7), turned to 0 degrees
- moved C76 341.2 mm to (130.4, 123.0), turned to 0 degrees
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
Commit message: fix: update power symbol and reference designators in ECU schematic and PCB files
Connections:
- K20 pad 14: +12V -> +BAT
Changed lines of the file:
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@@
 			(layers "*.Cu" "*.Mask")
 			(remove_unused_layers no)
-			(net "+12V")
+			(net "+BAT")
 			(pintype "passive")
 		)

Commit message: fix: update net name from "+BAT" to "+12V" in ECU PCB file
Connections:
- J7 pad 12: +BAT -> +12V
Changed lines of the file:
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@@
 			(layers "*.Cu" "*.Mask")
 			(remove_unused_layers no)
-			(net "+BAT")
+			(net "+12V")
 			(pinfunction "12_12")
 			(pintype "passive")

Commit message: Enhance ECU design files with updated parameters and new libraries
- Updated `ecu.kicad_pro` with new zone parameters, track widths, and DRC rules to improve design flexibility and manufacturability.
- Added `erc_report.json` to capture electrical rule check results, including warnings for multiple net names.
- Introduced `fp-lib-table` and `sym-lib-table` to include project-local libraries for footprints and symbols, enhancing design organization and accessibility.
Parts:
- D1: value ESDALC6V1-1U2 -> PESD5V0S1BA,115; footprint Diode_SMD:Infineon_SG-WLL-2-3_0.58x0.28_P0.36mm -> Diode_SMD:D_SOD-323
- D19, D20: footprint LED_SMD:LED_0201_0603Metric -> LED_SMD:LED_0603_1608Metric
- T201: value KMS-1102NL -> SM91071AL-E; footprint Transformer_SMD:Transformer_Pulse_H1100NL -> Starlight:Bourns_SM91071AL-E
- U4: footprint Package_DFN_QFN:VQFN-24-1EP_4x4mm_P0.5mm_EP2.5x2.5mm_ThermalVias -> Starlight:VQFN-24-1EP_4x4mm_P0.5mm_EP2.5x2.5mm_POFV
- moved K18 57.5 mm to (203.3, 174.0)
- moved K21 57.5 mm to (169.3, 200.5)
- moved K27 53.0 mm to (237.3, 200.5)
- moved K23 51.0 mm to (186.3, 200.5)
- moved K14 43.1 mm to (152.3, 200.5)
- moved K24 43.1 mm to (237.3, 147.5)
- moved K26 34.0 mm to (220.3, 200.5)
- moved K13 31.5 mm to (203.3, 121.0)
- moved K17 31.5 mm to (186.3, 174.0)
- moved K20 31.5 mm to (220.3, 147.5)
- moved K22 26.5 mm to (220.3, 174.0)
- moved K19 17.0 mm to (203.3, 147.5)
- moved K3 17.0 mm to (186.3, 147.5)
- moved D20 14.2 mm to (277.0, 124.4)
- moved D19 13.5 mm to (273.8, 124.4)
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
Commit message: feat: update ECU 4-layer layout and fabrication profile
Parts:
- moved U302 141.1 mm to (145.8, 239.1), turned to 0 degrees
- moved U301 140.2 mm to (125.8, 239.1), turned to 0 degrees
- moved C5 128.6 mm to (133.3, 236.6), turned to -90 degrees
- moved K26 122.6 mm to (132.0, 115.5)
- moved C67 118.6 mm to (173.3, 236.6), turned to -90 degrees
- moved C66 115.8 mm to (153.3, 236.6), turned to -90 degrees
- moved C10 109.8 mm to (336.1, 68.3)
- moved C11 109.8 mm to (332.8, 78.0)
- moved C12 109.8 mm to (336.1, 78.0)
- moved C13 109.8 mm to (332.1, 70.9)
- moved C14 109.8 mm to (332.1, 74.2)
- moved C15 109.8 mm to (338.6, 80.6)
- moved C19 109.8 mm to (357.1, 70.0)
- moved C20 109.8 mm to (357.1, 78.8)
- moved C23 109.8 mm to (351.6, 82.8)
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Connections:
- J6 pad 1: /06_Relay_Matrix/VIB_ENABLE_DEVICE_SIDE -> /06_Relay_Matrix/ENGINE_START_DEVICE_SIDE
- J6 pad 10: /06_Relay_Matrix/PUMP1_DEVICE_SIDE -> /06_Relay_Matrix/FRONT_LED_HEADLAMP_DEVICE_SIDE
- J6 pad 11: /06_Relay_Matrix/ENGINE_START_DEVICE_SIDE -> /06_Relay_Matrix/HORN_DEVICE_SIDE
- J6 pad 12: /06_Relay_Matrix/FRONT_LED_HEADLAMP_DEVICE_SIDE -> /06_Relay_Matrix/VIB_ENABLE_DEVICE_SIDE
- J6 pad 13: /06_Relay_Matrix/FRONT_MAIN_LAMP_DEVICE_SIDE -> /06_Relay_Matrix/TRAVEL_SPEED_RANGE_DEVICE_SIDE
- J6 pad 14: /06_Relay_Matrix/LEFT_TURN_SIGNAL_DEVICE_SIDE -> /06_Relay_Matrix/PUMP2_DEVICE_SIDE
- J6 pad 15: unconnected-(J6-Pad15) -> /06_Relay_Matrix/RIGHT_TURN_SIGNAL_DEVICE_SIDE
- J6 pad 16: unconnected-(J6-Pad16) -> /06_Relay_Matrix/E_STOP_DEVICE_SIDE
- J6 pad 17: +12V -> /06_Relay_Matrix/ENGINE_SPEED_OEM_SIDE
- J6 pad 18: +12V -> /06_Relay_Matrix/PARK_BRAKE_DEVICE_SIDE
- J6 pad 19: /06_Relay_Matrix/VIB_ENABLE_OEM_SIDE -> /06_Relay_Matrix/VIB_REAR_DEVICE_SIDE
- J6 pad 2: /06_Relay_Matrix/VIB_HIGH_DEVICE_SIDE -> /06_Relay_Matrix/TRAVEL_SPEED_RANGE_OEM_SIDE
- J6 pad 20: /06_Relay_Matrix/VIB_HIGH_OEM_SIDE -> /06_Relay_Matrix/REAR_LED_HEADLAMP_DEVICE_SIDE
- J6 pad 21: /06_Relay_Matrix/VIB_LOW_OEM_SIDE -> /06_Relay_Matrix/PUMP1_DEVICE_SIDE
- J6 pad 22: /06_Relay_Matrix/VIB_FRONT_OEM_SIDE -> /06_Relay_Matrix/VIB_ENABLE_OEM_SIDE
- J6 pad 23: /06_Relay_Matrix/VIB_REAR_OEM_SIDE -> /06_Relay_Matrix/VIB_FRONT_OEM_SIDE
- J6 pad 24: /06_Relay_Matrix/ENGINE_SPEED_OEM_SIDE -> /06_Relay_Matrix/VIB_LOW_DEVICE_SIDE
- J6 pad 25: /06_Relay_Matrix/TRAVEL_SPEED_RANGE_OEM_SIDE -> /06_Relay_Matrix/VIB_HIGH_DEVICE_SIDE
- J6 pad 26: /06_Relay_Matrix/PARK_BRAKE_OEM_SIDE -> +12V
- J6 pad 27: /06_Relay_Matrix/E_STOP_OEM_SIDE -> +12V
- J6 pad 28: /06_Relay_Matrix/PUMP2_DEVICE_SIDE -> /07_Valve/YV_FWD_COIL_N
- J6 pad 29: /06_Relay_Matrix/HORN_DEVICE_SIDE -> /07_Valve/YV_BACK_COIL_N
- J6 pad 3: /06_Relay_Matrix/VIB_LOW_DEVICE_SIDE -> /06_Relay_Matrix/FRONT_MAIN_LAMP_DEVICE_SIDE
- J6 pad 30: /06_Relay_Matrix/REVERSE_ALARM_DEVICE_SIDE -> unconnected-(J6-Pad30)
- J6 pad 31: /06_Relay_Matrix/REAR_LED_HEADLAMP_DEVICE_SIDE -> unconnected-(J6-Pad31)
- J6 pad 32: /06_Relay_Matrix/REAR_MAIN_LAMP_DEVICE_SIDE -> /06_Relay_Matrix/E_STOP_OEM_SIDE
- J6 pad 33: /06_Relay_Matrix/RIGHT_TURN_SIGNAL_DEVICE_SIDE -> /06_Relay_Matrix/VIB_LOW_OEM_SIDE
- J6 pad 34: /07_Valve/YV_FWD_COIL_N -> /06_Relay_Matrix/VIB_HIGH_OEM_SIDE
- J6 pad 35: /07_Valve/YV_BACK_COIL_N -> /06_Relay_Matrix/VIB_FRONT_DEVICE_SIDE
- J6 pad 4: /06_Relay_Matrix/VIB_FRONT_DEVICE_SIDE -> /06_Relay_Matrix/ENGINE_SPEED_DEVICE_SIDE
- J6 pad 5: /06_Relay_Matrix/VIB_REAR_DEVICE_SIDE -> /06_Relay_Matrix/LEFT_TURN_SIGNAL_DEVICE_SIDE
- J6 pad 6: /06_Relay_Matrix/ENGINE_SPEED_DEVICE_SIDE -> /06_Relay_Matrix/PARK_BRAKE_OEM_SIDE
- J6 pad 7: /06_Relay_Matrix/TRAVEL_SPEED_RANGE_DEVICE_SIDE -> /06_Relay_Matrix/REVERSE_ALARM_DEVICE_SIDE
- J6 pad 8: /06_Relay_Matrix/PARK_BRAKE_DEVICE_SIDE -> /06_Relay_Matrix/REAR_MAIN_LAMP_DEVICE_SIDE
- J6 pad 9: /06_Relay_Matrix/E_STOP_DEVICE_SIDE -> /06_Relay_Matrix/VIB_REAR_OEM_SIDE
Routing:
- net /06_Relay_Matrix/VIB_HIGH_DEVICE_SIDE: track 0.00 -> 252.8 mm
- net /06_Relay_Matrix/VIB_LOW_DEVICE_SIDE: track 0.00 -> 207.9 mm
- net /06_Relay_Matrix/VIB_LOW_OEM_SIDE: track 0.00 -> 172.3 mm, vias 0 -> 1
- net /06_Relay_Matrix/TRAVEL_SPEED_RANGE_DEVICE_SIDE: track 0.00 -> 168.9 mm
- net /06_Relay_Matrix/VIB_HIGH_OEM_SIDE: track 0.00 -> 142.5 mm, vias 0 -> 1
- net /06_Relay_Matrix/TRAVEL_SPEED_RANGE_OEM_SIDE: track 0.00 -> 116.8 mm
- net /06_Relay_Matrix/VIB_FRONT_DEVICE_SIDE: track 0.00 -> 113.1 mm
- net /06_Relay_Matrix/ENGINE_SPEED_DEVICE_SIDE: track 0.00 -> 102.3 mm
- net /06_Relay_Matrix/VIB_FRONT_OEM_SIDE: track 0.00 -> 91.9 mm
- net /06_Relay_Matrix/VIB_REAR_DEVICE_SIDE: track 0.00 -> 86.3 mm
- net /06_Relay_Matrix/ENGINE_START_DEVICE_SIDE: track 0.00 -> 81.2 mm
- net /06_Relay_Matrix/ENGINE_SPEED_OEM_SIDE: track 0.00 -> 80.8 mm
- net /06_Relay_Matrix/RIGHT_TURN_SIGNAL_DEVICE_SIDE: track 0.00 -> 79.1 mm
- net /06_Relay_Matrix/VIB_ENABLE_DEVICE_SIDE: track 0.00 -> 76.6 mm
- net /06_Relay_Matrix/VIB_REAR_OEM_SIDE: track 0.00 -> 69.9 mm
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- added copper zone on In2.Cu, net +BAT
- added copper zone on In1.Cu, net PGND
Other:
- rule solder_mask_min_width: 0.12 -> 0.2

Commit message: Refactor ECU schematic: Adjust wire connections and update no_connect points
- Modified coordinates for several no_connect points to improve layout clarity.
- Adjusted wire connections to reflect updated schematic design.
- Removed redundant wire segments and ensured UUIDs are consistent with changes.
- Enhanced overall readability and organization of the schematic for better maintenance.
Parts:
- moved D2 183.7 mm to (244.2, 126.0)
- moved R1 183.7 mm to (241.2, 134.3)
- moved R79 183.7 mm to (251.5, 120.6)
- moved U11 183.7 mm to (270.0, 117.0)
- moved C72 183.7 mm to (240.8, 139.2)
- moved C73 183.7 mm to (244.1, 139.2)
- moved C74 183.7 mm to (247.4, 130.5)
- moved C75 183.7 mm to (258.0, 139.2)
- moved C76 183.7 mm to (261.3, 139.2)
- moved C77 183.7 mm to (264.6, 130.5)
- moved D3 183.7 mm to (261.4, 126.0)
- moved Q2 183.7 mm to (245.7, 118.8)
- moved Q3 183.7 mm to (262.9, 118.8)
- moved R2 183.7 mm to (258.4, 134.3)
- moved R80 183.7 mm to (253.3, 120.6)
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Connections:
- K1 pad A2: /05_Relay_Drivers/DTAIN22 -> /05_Relay_Drivers/DTAIN03
- K10 pad A2: /05_Relay_Drivers/DTAIN31 -> /05_Relay_Drivers/DTAIN23
- K11 pad A2: /05_Relay_Drivers/DTAIN11 -> /05_Relay_Drivers/DTAIN25
- K12 pad A2: /05_Relay_Drivers/DTAIN04 -> /05_Relay_Drivers/DTAIN26
- K13 pad A2: /05_Relay_Drivers/DTAIN20 -> /05_Relay_Drivers/DTAIN32
- K14 pad A2: /05_Relay_Drivers/DTAIN21 -> /05_Relay_Drivers/DTAIN31
- K15 pad A2: /05_Relay_Drivers/DTAIN05 -> /05_Relay_Drivers/DTAIN07
- K16 pad A2: /05_Relay_Drivers/DTAIN14 -> /05_Relay_Drivers/DTAIN17
- K17 pad A2: /05_Relay_Drivers/DTAIN16 -> /05_Relay_Drivers/DTAIN24
- K18 pad A2: /05_Relay_Drivers/DTAIN10 -> /05_Relay_Drivers/DTAIN27
- K19 pad A2: /05_Relay_Drivers/DTAIN17 -> /05_Relay_Drivers/DTAIN34
- K2 pad A2: /05_Relay_Drivers/DTAIN26 -> /05_Relay_Drivers/DTAIN01
- K20 pad A2: /05_Relay_Drivers/DTAIN03 -> /05_Relay_Drivers/DTAIN37
- K21 pad A2: /05_Relay_Drivers/DTAIN07 -> /05_Relay_Drivers/DTAIN02
- K22 pad A2: /05_Relay_Drivers/DTAIN06 -> /05_Relay_Drivers/DTAIN35
- K23 pad A2: /05_Relay_Drivers/DTAIN15 -> /05_Relay_Drivers/DTAIN16
- K24 pad A2: /05_Relay_Drivers/DTAIN02 -> /05_Relay_Drivers/DTAIN33
- K25 pad A2: /05_Relay_Drivers/DTAIN00 -> /05_Relay_Drivers/DTAIN30
- K26 pad A2: /05_Relay_Drivers/DTAIN12 -> /05_Relay_Drivers/DTAIN06
- K27 pad A2: /05_Relay_Drivers/DTAIN13 -> /05_Relay_Drivers/DTAIN36
- K3 pad A2: /05_Relay_Drivers/DTAIN01 -> /05_Relay_Drivers/DTAIN20
- K4 pad A2: /05_Relay_Drivers/DTAIN25 -> /05_Relay_Drivers/DTAIN11
- K5 pad A2: /05_Relay_Drivers/DTAIN30 -> /05_Relay_Drivers/DTAIN22
- K6 pad A2: /05_Relay_Drivers/DTAIN27 -> /05_Relay_Drivers/DTAIN21
- K7 pad A2: /05_Relay_Drivers/DTAIN24 -> /05_Relay_Drivers/DTAIN04
- K8 pad A2: /05_Relay_Drivers/DTAIN23 -> /05_Relay_Drivers/DTAIN00
- K9 pad A2: /05_Relay_Drivers/DTAIN32 -> /05_Relay_Drivers/DTAIN10
Routing:
- net /05_Relay_Drivers/TPIC5_CLR_N: track 0.00 -> 135.4 mm, vias 0 -> 5
- net /05_Relay_Drivers/TPIC5_OE_N: track 0.00 -> 133.1 mm, vias 0 -> 5
- net /05_Relay_Drivers/DTAIN36: track 0.00 -> 132.3 mm
- net /05_Relay_Drivers/DTAIN35: track 0.00 -> 125.8 mm
- net /05_Relay_Drivers/DTAIN26: track 0.00 -> 122.4 mm, vias 0 -> 2
- net /05_Relay_Drivers/DTAIN16: track 0.00 -> 121.7 mm, vias 0 -> 2
- net /05_Relay_Drivers/DTAIN06: track 0.00 -> 119.1 mm, vias 0 -> 2
- net /05_Relay_Drivers/DTAIN25: track 0.00 -> 113.9 mm
- net /07_Valve/YV_BACK_COIL_N: track 0.00 -> 111.1 mm, vias 0 -> 2
- net /05_Relay_Drivers/TPIC5_RCK: track 0.00 -> 110.2 mm, vias 0 -> 5
- net /05_Relay_Drivers/TPIC5_SER: track 0.00 -> 108.7 mm, vias 0 -> 3
- net /05_Relay_Drivers/TPIC5_SRCK: track 0.00 -> 106.6 mm, vias 0 -> 5
- net /05_Relay_Drivers/DTAIN37: track 0.00 -> 105.9 mm
- net /07_Valve/YV_FWD_COIL_N: track 0.00 -> 105.4 mm, vias 0 -> 2
- net GND: track 0.00 -> 103.2 mm, vias 0 -> 5
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- added copper zone on F.Cu, net +12V
- added copper zone on In2.Cu, net +12V
- added copper zone on F.Cu, net +BAT
- added copper zone on F.Cu, net PGND

Commit message: Implement code changes to enhance functionality and improve performance
Parts:
- moved U12 42.6 mm to (227.2, 119.9), turned to 0 degrees
- moved D3 38.6 mm to (227.1, 108.2), turned to -90 degrees
- moved C77 38.0 mm to (227.2, 123.5), turned to 180 degrees
- moved R83 37.6 mm to (233.2, 115.2), turned to 0 degrees
- moved U11 36.8 mm to (233.2, 118.1), turned to 90 degrees
- moved R2 36.6 mm to (227.2, 115.1), turned to 180 degrees
- moved R84 36.3 mm to (236.4, 115.2), turned to 0 degrees
- moved C76 33.4 mm to (233.2, 121.0)
- moved R82 32.9 mm to (235.8, 118.4), turned to -90 degrees
- moved Q3 30.1 mm to (234.8, 108.0), turned to 90 degrees
- moved C75 29.8 mm to (233.2, 122.6)
- moved R1 19.2 mm to (242.3, 115.1), turned to 180 degrees
- moved C73 18.6 mm to (248.2, 121.0)
- moved D2 17.9 mm to (242.4, 108.2), turned to -90 degrees
- moved C72 15.7 mm to (242.0, 123.5), turned to 180 degrees
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Routing:
- net PGND: track 39.8 -> 65.7 mm, vias 83 -> 89
- net /07_Valve/YV_FWD_COIL_N: track 105.4 -> 129.1 mm, vias 2 -> 5
- net GND: track 103.2 -> 123.1 mm
- net Net-(D3-A): track 0.00 -> 18.6 mm
- net Net-(D2-A): track 0.00 -> 18.5 mm
- net +3.3V: track 0.00 -> 8.68 mm
- net /07_Valve/YV_BACK_COIL_N: track 111.1 -> 119.1 mm, vias 2 -> 5
- net +5V: track 86.5 -> 93.3 mm
- net Net-(Q2-G): track 0.00 -> 4.39 mm
- net Net-(Q3-G): track 0.00 -> 4.38 mm
- net Net-(U11-OUT): track 0.00 -> 1.81 mm
- net Net-(U10-OUT): track 0.00 -> 1.81 mm
- net Net-(U11-IN+): track 0.00 -> 1.66 mm
- net Net-(U10-IN+): track 0.00 -> 1.66 mm
- added copper zone on F.Cu, net /07_Valve/YV_BACK_COIL_N
- added copper zone on F.Cu, net /07_Valve/YV_FWD_COIL_N

Commit message: Refactor QFN-234MMX5MM_MPQ4371_MNP footprint: Update pad definitions to custom shapes with mesh-connect lands, adjust silk layer properties, and enhance pad geometries for improved thermal performance.
Parts:
- moved R58 61.4 mm to (302.2, 91.8)
- moved C52 61.4 mm to (302.2, 94.1)
- moved C53 61.4 mm to (305.5, 94.1)
- moved C54 61.4 mm to (318.2, 71.3)
- moved C55 61.4 mm to (318.2, 73.1)
- moved C56 61.4 mm to (318.2, 74.9)
- moved C57 61.4 mm to (318.2, 76.7)
- moved C58 61.4 mm to (318.2, 78.5)
- moved C59 61.4 mm to (318.2, 80.4)
- moved C60 61.4 mm to (313.5, 86.9)
- moved C61 61.4 mm to (315.3, 86.9)
- moved C62 61.4 mm to (317.1, 86.9)
- moved C63 61.4 mm to (318.9, 86.9)
- moved C64 61.4 mm to (301.4, 83.1)
- moved C65 61.4 mm to (303.2, 83.1)
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