File: pcb/roller/ecu/03_Ethernet.kicad_sch (KiCad schematic)
At the start: 44 parts, among them J3 SS-12400-004, T201 KMS-1102NL, U4 LAN8742A, U5 USBLC6-4SC6, Y3 25MHz

Commit message: Add power symbols for +1V0 and PWR_FLAG to the schematic
- Introduced a new global power symbol for +1V0 with appropriate properties and pin configurations.
- Added a PWR_FLAG symbol to indicate power source in the schematic, enhancing ERC capabilities.
- Updated the used designators in the project file to include new power symbols.
Connections:
- net +3V3_ETH: now reaches C58.1, C59.1, C60.1, C61.1, C62.1, C63.1, FB1.2, R58.2, R59.2, R67.2, R68.2, T201.2 (TX_CT), T201.7 (RX_CT), U4.1 (VDD2A), U4.19 (VDD1A), U5.5 (VBUS)
Other:
- note added: "Internal 1.2 V regulator enabled"

Commit message: Add design settings and DRC rules to ECU PCB configuration
- Introduced comprehensive design settings including defaults for various parameters such as line widths, text sizes, and pad dimensions.
- Added detailed DRC (Design Rule Check) exclusions and rule severities to enhance error handling and warnings during PCB design.
- Updated tuning pattern settings and teardrop parameters for improved track and pad connections.
- Cleared previously used designators for better organization and clarity in the design file.
Parts:
- T201: symbol ECU_Custom:KMS-1102NL -> Starlight:KMS-1102NL
Other:
- note added: "PA1"
- note added: "PA2"
- note added: "PA7"
- note added: "PB14"
- note added: "PB15"
- note added: "PC1"
- note added: "PC4"
- note added: "PC5"
- note added: "PG11"
- note added: "PG13"

Commit message: Enhance ECU design files with updated parameters and new libraries
- Updated `ecu.kicad_pro` with new zone parameters, track widths, and DRC rules to improve design flexibility and manufacturability.
- Added `erc_report.json` to capture electrical rule check results, including warnings for multiple net names.
- Introduced `fp-lib-table` and `sym-lib-table` to include project-local libraries for footprints and symbols, enhancing design organization and accessibility.
Parts:
- D19, D20: footprint LED_SMD:LED_0201_0603Metric -> LED_SMD:LED_0603_1608Metric
- T201: value KMS-1102NL -> SM91071AL-E; footprint Transformer_SMD:Transformer_Pulse_H1100NL -> Starlight:Bourns_SM91071AL-E; symbol Starlight:KMS-1102NL -> Starlight:SM91071AL-E
- U4: footprint Package_DFN_QFN:VQFN-24-1EP_4x4mm_P0.5mm_EP2.5x2.5mm_ThermalVias -> Starlight:VQFN-24-1EP_4x4mm_P0.5mm_EP2.5x2.5mm_POFV
Changed lines of the file:
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@@
 	)
 	(symbol
-		(lib_id "Starlight:KMS-1102NL")
+		(lib_id "Starlight:SM91071AL-E")
 		(at 218.44 85.09 0)
 		(unit 1)
@@
 			)
 		)
-		(property "Value" "KMS-1102NL"
+		(property "Value" "SM91071AL-E"
 			(at 210.312 73.66 0)
 			(show_name no)
@@
 			)
 		)
-		(property "Footprint" "Transformer_SMD:Transformer_Pulse_H1100NL"
+		(property "Footprint" "Starlight:Bourns_SM91071AL-E"
 			(at 218.44 85.09 0)
 			(hide yes)
@@
 			)
 		)
-		(property "Footprint" "LED_SMD:LED_0201_0603Metric"
+		(property "Footprint" "LED_SMD:LED_0603_1608Metric"
 			(at 180.34 130.81 0)
 			(hide yes)
@@
 			)
 		)
-		(property "Footprint" "LED_SMD:LED_0201_0603Metric"
+		(property "Footprint" "LED_SMD:LED_0603_1608Metric"
 			(at 162.56 130.81 0)
 			(hide yes)
@@
 			)
 		)
-		(property "Footprint" "Package_DFN_QFN:VQFN-24-1EP_4x4mm_P0.5mm_EP2.5x2.5mm_ThermalVias"
+		(property "Footprint" "Starlight:VQFN-24-1EP_4x4mm_P0.5mm_EP2.5x2.5mm_POFV"
 			(at 128.27 118.11 0)
 			(hide yes)

Commit message: Update used_designators in ecu.kicad_pro to include resistors R113-115
Parts:
- added R113, R114, R115: 33R, Resistor_SMD:R_0603_1608Metric, symbol Device:R
Connections:
- net RMII_TXD0: now also R113.1; no longer U4.17 (TXD0)
- net RMII_TXD1: now also R114.1; no longer U4.18 (TXD1)
- net RMII_TX_EN: now also R115.1; no longer U4.16 (TXEN)
- new net: R114.2, U4.18 (TXD1)
- new net: R113.2, U4.17 (TXD0)
- new net: R115.2, U4.16 (TXEN)
